Commit message: added left and right wheel to base link - urdf

File: urdf/clubbot.urdf (robot description, URDF)
Before this commit: robot ClubBotII, 2 links, 1 joints
Links:
- added link right_wheel, mass 0.055; collision cylinder length=0.04 radius=0.04; visual mesh filename=package://clubbot_description/meshes/SpikeyWheel.stl scale=0.001 0.001 0.001
Joints:
- added joint right_wheel_to_base_link: type continuous, parent base_link, child right_wheel, origin xyz=-0.09 0.01 -0.05 rpy=0 -1.5708 0, axis 0 0 1
- joint left_wheel_to_base_link: origin xyz=0 0.0 0.0 -> xyz=0.09 0.01 -0.05 rpy=0 1.5708 0

Commit message: added usb camera top - urdf

File: urdf/clubbot.urdf (robot description, URDF)
Before this commit: robot ClubBotII, 3 links, 2 joints
Links:
- added link top_usb_cam; visual mesh filename=package://clubbot_description/meshes/camera_top.stl scale=0.001 0.001 0.001
Joints:
- added joint top_to_base: type fixed, parent base_link, child top_usb_cam, origin xyz=-0.00 0.00 0.05 rpy=0 0 0
